File: Routage_H2O_Laurie_v1.kicad_pcb (KiCad board)
At the start: 2 copper layers, 110 x 100 mm, 52 parts, among them J2 Conn_01x02, J3 Conn_01x03, Q1 2N2907, Q10 TIP32, Q11 BD138, Q12 TIP31, Q13 2N2222, Q2 2N2907, Q3 2N2907, Q4 2N2222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

Commit message: crashtest
Parts:
- moved R13 48.6 mm to (133.3, 27.9)
- moved C7 43.2 mm to (190.5, 76.2), turned to 0 degrees
- moved C4 40.4 mm to (91.4, 64.8), turned to 0 degrees
- moved C6 30.5 mm to (190.5, 67.3), turned to 0 degrees
- moved C5 29.9 mm to (102.9, 67.3), turned to 90 degrees
- moved C8 29.7 mm to (95.2, 39.4), turned to 0 degrees
- moved Q9 27.4 mm to (109.2, 68.6), turned to 0 degrees
- moved C10 23.2 mm to (184.2, 38.1), turned to 0 degrees
- moved Q13 20.5 mm to (146.1, 57.1), turned to 0 degrees
- moved J3 20.3 mm to (127.0, 30.5)
- moved R11 17.8 mm to (108.0, 41.9)
- moved D2 15.2 mm to (138.4, 52.1), turned to 270 degrees
- moved R16 14.9 mm to (133.3, 49.5), turned to 270 degrees
- moved C9 14.5 mm to (100.3, 29.2)
- moved J2 14.0 mm to (163.8, 30.5)
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