File: Routage_H2O_Laurie_v1.sch (KiCad schematic (older format))
At the start: 52 parts, among them J2 Conn_01x02, J3 Conn_01x03, Q1 2N2907, Q10 TIP32, Q11 BD138, Q12 TIP31, Q13 2N2222, Q2 2N2907, Q3 2N2907, Q4 2N2222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

Commit message: crashtest
Parts:
- U1: symbol CmpAmpliAudio:Relay_1CT -> Routage_H2O_Laurie_v1-rescue:Relay_1CT-CmpAmpliAudio
- U2: symbol CmpAmpliAudio:Jack_Mono -> Routage_H2O_Laurie_v1-rescue:Jack_Mono-CmpAmpliAudio
Changed lines of the file:
@@
 	8300 2850 8300 5850
 $Comp
-L CmpAmpliAudio:Jack_Mono U2
+L Routage_H2O_Laurie_v1-rescue:Jack_Mono-CmpAmpliAudio U2
 U 1 1 605BBF3F
 P 1000 3800
@@
 	1200 3900 1500 3900
 $Comp
-L CmpAmpliAudio:Relay_1CT U1
+L Routage_H2O_Laurie_v1-rescue:Relay_1CT-CmpAmpliAudio U1
 U 1 1 605CF78D
 P 9800 2750

Commit message: PlacementFinito
Parts:
- added D3, D4: 1N4001, LibAmpli_3imacs:D_DO-35_SOD27_P10.16mm_Horizontal, symbol Device:D
Connections:
- net +12V: now also D3.1 (K)
- net -12V: now also D4.2 (A)
- net GND: now also D3.2 (A), D4.1 (K)
- no-connect marks 0 -> 1
Changed lines of the file:
@@
 L power:GND #PWR018
 U 1 1 60840977
-P 2500 6850
-F 0 "#PWR018" H 2500 6600 50  0001 C CNN
-F 1 "GND" H 2505 6677 50  0000 C CNN
-F 2 "" H 2500 6850 50  0001 C CNN
-F 3 "" H 2500 6850 50  0001 C CNN
-	1    2500 6850
-	1    0    0    -1
-$EndComp
-Wire Wire Line
-	2500 6700 2500 6850
+P 2850 6850
+F 0 "#PWR018" H 2850 6600 50  0001 C CNN
+F 1 "GND" H 2855 6677 50  0000 C CNN
+F 2 "" H 2850 6850 50  0001 C CNN
+F 3 "" H 2850 6850 50  0001 C CNN
+	1    2850 6850
+	1    0    0    -1
+$EndComp
+Wire Wire Line
+	2850 6700 2850 6850
 $Comp
 L Connector_Generic:Conn_01x03 J3
@@
 	1350 6700 1750 6700
 Wire Wire Line
-	2100 6700 2500 6700
-Wire Wire Line
 	1750 6700 2100 6700
 Wire Wire Line
@@
 Wire Wire Line
 	1550 6000 1550 6100
+Wire Wire Line
+	2100 6700 2500 6700
+$Comp
+L Device:D D3
+U 1 1 6074947E
+P 2500 6350
+F 0 "D3" V 2454 6430 50  0000 L CNN
+F 1 "1N4001" V 2545 6430 50  0000 L CNN
+F 2 "LibAmpli_3imacs:D_DO-35_SOD27_P10.16mm_Horizontal" H 2500 6350 50  0001 C CNN
+F 3 "~" H 2500 6350 50  0001 C CNN
+	1    2500 6350
+	0    1    1    0
+$EndComp
+$Comp
+L Device:D D4
+U 1 1 6074B471
+P 2500 7100
+F 0 "D4" V 2454 7180 50  0000 L CNN
+F 1 "1N4001" V 2545 7180 50  0000 L CNN
+F 2 "LibAmpli_3imacs:D_DO-35_SOD27_P10.16mm_Horizontal" H 2500 7100 50  0001 C CNN
+F 3 "~" H 2500 7100 50  0001 C CNN
+	1    2500 7100
+	0    1    1    0
+$EndComp
+Wire Wire Line
+	2100 6100 2500 6100
+Wire Wire Line
+	2500 6100 2500 6200
+Connection ~ 2100 6100
+Wire Wire Line
+	2500 6500 2500 6700
+Connection ~ 2500 6700
+Wire Wire Line
+	2500 6700 2850 6700
+Wire Wire Line
+	2500 6950 2500 6700
+Wire Wire Line
+	2100 7350 2500 7350
+Wire Wire Line
+	2500 7350 2500 7250
+Connection ~ 2100 7350
+NoConn ~ 1200 3800
 $EndSCHEMATC
